Commit message: Add files via upload

File: description/right_arm.xacro (robot description, xacro)
@@ -3,44 +3,44 @@
     <!--3 juntas ombro + 2 juntas cotovelo + 2 mao + 1 garra __ 7DOF-->
     <!--SHOULDER-ELBOW-->
-    <joint name="L_shoulder_joint" type="fixed">
+    <joint name="R_shoulder_joint" type="fixed">
         <parent link="body_link"/>
-        <child link="L_shoulder_aux_link"/>
-        <origin xyz="0.05 0.13 1.05" rpy="0 0 0"/>
-    </joint>
-    <link name="L_shoulder_aux_link">
-        <xacro:inertial_box mass="0.1" x="0" y="0" z="0">
-            <origin xyz="0 0 0" rpy="0 0 0"/>
-        </xacro:inertial_box>
-    </link>
-    <joint name="L_shoulder_joint_y" type="revolute">
-        <parent link="L_shoulder_aux_link"/>
-        <child link="L_shoulder_link_y"/>
-        <origin xyz="0 0 0" rpy="0 0 0"/>
-        <axis xyz="1 0 0"/>
+        <child link="R_shoulder_aux_link"/>
+        <origin xyz="0.05 -0.13 1.05" rpy="0 0 0"/>
+    </joint>
+    <link name="R_shoulder_aux_link">
+        <xacro:inertial_box mass="0.1" x="0" y="0" z="0">
+            <origin xyz="0 0 0" rpy="0 0 0"/>
+        </xacro:inertial_box>
+    </link>
+    <joint name="R_shoulder_joint_y" type="revolute">
+        <parent link="R_shoulder_aux_link"/>
+        <child link="R_shoulder_link_y"/>
+        <origin xyz="0 0 0" rpy="0 0 0"/>
+        <axis xyz="-1 0 0"/>
         <limit effort="1000.0" lower="0" upper="0.785" velocity="0.5"/>
     </joint>
-    <link name="L_shoulder_link_y">
-        <xacro:inertial_box mass="0.1" x="0" y="0" z="0">
-            <origin xyz="0 0 0" rpy="0 0 0"/>
-        </xacro:inertial_box>
-    </link>
-    <joint name="L_shoulder_joint_x" type="revolute">
-        <parent link="L_shoulder_link_y"/>
-        <child link="L_shoulder_link_x"/>
+    <link name="R_shoulder_link_y">
+        <xacro:inertial_box mass="0.1" x="0" y="0" z="0">
+            <origin xyz="0 0 0" rpy="0 0 0"/>
+        </xacro:inertial_box>
+    </link>
+    <joint name="R_shoulder_joint_x" type="revolute">
+        <parent link="R_shoulder_link_y"/>
+        <child link="R_shoulder_link_x"/>
         <origin xyz="0 0 0" rpy="0 0 0"/>
         <axis xyz="0 -1 0"/>
         <limit effort="1000.0" lower="-0.785" upper="2.356" velocity="0.5"/>
     </joint>
-    <link name="L_shoulder_link_x">
-        <xacro:inertial_box mass="0.1" x="0" y="0" z="0">
-            <origin xyz="0 0 0" rpy="0 0 0"/>
-        </xacro:inertial_box>
-    </link>
-    <joint name="L_shoulder_final_joint" type="fixed">
-        <parent link="L_shoulder_link_x"/>
-        <child link="L_shoulder_link"/>
-        <origin xyz="0 0 0" rpy="0 0 0"/>
-    </joint>
-    <link name="L_shoulder_link">
+    <link name="R_shoulder_link_x">
+        <xacro:inertial_box mass="0.1" x="0" y="0" z="0">
+            <origin xyz="0 0 0" rpy="0 0 0"/>
+        </xacro:inertial_box>
+    </link>
+    <joint name="R_shoulder_final_joint" type="fixed">
+        <parent link="R_shoulder_link_x"/>
+        <child link="R_shoulder_link"/>
+        <origin xyz="0 0 0" rpy="0 0 0"/>
+    </joint>
+    <link name="R_shoulder_link">
         <visual>
             <origin xyz="0 0 -0.08" rpy="0 0 ${pi/2}"/>
@@ -60,14 +60,14 @@
         </xacro:inertial_box>
     </link>
-    <gazebo reference="L_shoulder_link">
+    <gazebo reference="R_shoulder_link">
         <material>Gazebo/Blue</material>
     </gazebo>
     <!--LIGAÇAO ELBOW-->
-    <joint name="L_shoulder_arm_joint" type="fixed">
-        <parent link="L_shoulder_link"/>
-        <child link="L_SE_link"/>
+    <joint name="R_shoulder_arm_joint" type="fixed">
+        <parent link="R_shoulder_link"/>
+        <child link="R_SE_link"/>
         <origin xyz="0 0 -0.2" rpy="0 0 0"/>
     </joint>
-    <link name="L_SE_link">
+    <link name="R_SE_link">
         <visual>
             <geometry>
@@ -85,48 +85,48 @@
         </xacro:inertial_sphere>
     </link>
-    <gazebo reference="L_SE_link">
+    <gazebo reference="R_SE_link">
         <material>Gazebo/Red</material>
     </gazebo>
     <!--ELBOW-WRIST-->
-    <joint name="L_elbow_joint" type="fixed">
-        <parent link="L_SE_link"/>
-        <child link="L_elbow_aux_link"/>
+    <joint name="R_elbow_joint" type="fixed">
+        <parent link="R_SE_link"/>
+        <child link="R_elbow_aux_link"/>
         <origin xyz="0 0 -0.04" rpy="0 0 0"/>
     </joint>
-    <link name="L_elbow_aux_link">
-        <xacro:inertial_box mass="0.1" x="0" y="0" z="0">
-            <origin xyz="0 0 0" rpy="0 0 0"/>
-        </xacro:inertial_box>
-    </link>
-    <joint name="L_elbow_joint_z" type="revolute">
-        <parent link="L_elbow_aux_link"/>
-        <child link="L_elbow_link_z"/>
-        <origin xyz="0 0 0" rpy="0 0 0"/>
-        <axis xyz="0 0 -1"/>
+    <link name="R_elbow_aux_link">
+        <xacro:inertial_box mass="0.1" x="0" y="0" z="0">
+            <origin xyz="0 0 0" rpy="0 0 0"/>
+        </xacro:inertial_box>
+    </link>
+    <joint name="R_elbow_joint_z" type="revolute">
+        <parent link="R_elbow_aux_link"/>
+        <child link="R_elbow_link_z"/>
+        <origin xyz="0 0 0" rpy="0 0 0"/>
+        <axis xyz="0 0 1"/>
         <limit effort="1000.0" lower="0" upper="1.445" velocity="0.5"/>
     </joint>
-    <link name="L_elbow_link_z">
-        <xacro:inertial_box mass="0.1" x="0" y="0" z="0">
-            <origin xyz="0 0 0" rpy="0 0 0"/>
-        </xacro:inertial_box>
-    </link>
-    <joint name="L_elbow_joint_x" type="revolute">
-        <parent link="L_elbow_link_z"/>
-        <child link="L_elbow_link_x"/>
+    <link name="R_elbow_link_z">
+        <xacro:inertial_box mass="0.1" x="0" y="0" z="0">
+            <origin xyz="0 0 0" rpy="0 0 0"/>
+        </xacro:inertial_box>
+    </link>
+    <joint name="R_elbow_joint_x" type="revolute">
+        <parent link="R_elbow_link_z"/>
+        <child link="R_elbow_link_x"/>
         <origin xyz="0 0 0" rpy="0 0 0"/>
         <axis xyz="0 -1 0"/>
         <limit effort="1000.0" lower="0" upper="2.225" velocity="0.5"/>
     </joint>
-    <link name="L_elbow_link_x">
-        <xacro:inertial_box mass="0.1" x="0" y="0" z="0">
-            <origin xyz="0 0 0" rpy="0 0 0"/>
-        </xacro:inertial_box>
-    </link>
-    <joint name="L_elbow_final_joint" type="fixed">
-        <parent link="L_elbow_link_x"/>
-        <child link="L_elbow_link"/>
-        <origin xyz="0 0 0" rpy="0 0 0"/>
-    </joint>
-    <link name="L_elbow_link">
+    <link name="R_elbow_link_x">
+        <xacro:inertial_box mass="0.1" x="0" y="0" z="0">
+            <origin xyz="0 0 0" rpy="0 0 0"/>
+        </xacro:inertial_box>
+    </link>
+    <joint name="R_elbow_final_joint" type="fixed">
+        <parent link="R_elbow_link_x"/>
+        <child link="R_elbow_link"/>
+        <origin xyz="0 0 0" rpy="0 0 0"/>
+    </joint>
+    <link name="R_elbow_link">
         <visual>
             <origin xyz="0 0 -0.08" rpy="0 0 ${pi/2}"/>
@@ -146,14 +146,14 @@
         </xacro:inertial_box>
     </link>
-    <gazebo reference="L_elbow_link">
+    <gazebo reference="R_elbow_link">
         <material>Gazebo/Blue</material>
     </gazebo>
     <!--LIGAÇAO WRIST-HAND-->
-    <joint name="L_WH_joint" type="fixed">
-        <parent link="L_elbow_link"/>
-        <child link="L_WH_link"/>
+    <joint name="R_WH_joint" type="fixed">
+        <parent link="R_elbow_link"/>
+        <child link="R_WH_link"/>
         <origin xyz="0 0 -0.2" rpy="0 0 0"/>
     </joint>
-    <link name="L_WH_link">
+    <link name="R_WH_link">
         <visual>
             <geometry>
@@ -171,48 +171,48 @@
         </xacro:inertial_sphere>
     </link>
-    <gazebo reference="L_WH_link">
+    <gazebo reference="R_WH_link">
         <material>Gazebo/Red</material>
     </gazebo>
     <!--HAND-->
-    <joint name="L_hand_joint" type="fixed">
-        <parent link="L_WH_link"/>
-        <child link="L_hand_aux_link"/>
+    <joint name="R_hand_joint" type="fixed">
+        <parent link="R_WH_link"/>
+        <child link="R_hand_aux_link"/>
         <origin xyz="0 0 -0.03" rpy="0 0 0"/>
     </joint>
-    <link name="L_hand_aux_link">
-        <xacro:inertial_box mass="0.1" x="0" y="0" z="0">
-            <origin xyz="0 0 0" rpy="0 0 0"/>
-        </xacro:inertial_box>
-    </link>
-    <joint name="L_hand_joint_z" type="revolute">
-        <parent link="L_hand_aux_link"/>
-        <child link="L_hand_link_z"/>
-        <origin xyz="0 0 0" rpy="0 0 0"/>
-        <axis xyz="0 0 -1"/>
+    <link name="R_hand_aux_link">
+        <xacro:inertial_box mass="0.1" x="0" y="0" z="0">
+            <origin xyz="0 0 0" rpy="0 0 0"/>
+        </xacro:inertial_box>
+    </link>
+    <joint name="R_hand_joint_z" type="revolute">
+        <parent link="R_hand_aux_link"/>
+        <child link="R_hand_link_z"/>
+        <origin xyz="0 0 0" rpy="0 0 0"/>
+        <axis xyz="0 0 1"/>
         <limit effort="1000.0" lower="-0.785" upper="0.785" velocity="0.5"/>
     </joint>
-    <link name="L_hand_link_z">
-        <xacro:inertial_box mass="0.1" x="0" y="0" z="0">
-            <origin xyz="0 0 0" rpy="0 0 0"/>
-        </xacro:inertial_box>
-    </link>
-    <joint name="L_hand_joint_x" type="revolute">
-        <parent link="L_hand_link_z"/>
-        <child link="L_hand_link_x"/>
+    <link name="R_hand_link_z">
+        <xacro:inertial_box mass="0.1" x="0" y="0" z="0">
+            <origin xyz="0 0 0" rpy="0 0 0"/>
+        </xacro:inertial_box>
+    </link>
+    <joint name="R_hand_joint_x" type="revolute">
+        <parent link="R_hand_link_z"/>
+        <child link="R_hand_link_x"/>
         <origin xyz="0 0 0" rpy="0 0 0"/>
         <axis xyz="0 -1 0"/>
         <limit effort="1000.0" lower="-0.785" upper="0.785" velocity="0.5"/>
     </joint>
-    <link name="L_hand_link_x">
-        <xacro:inertial_box mass="0.1" x="0" y="0" z="0">
-            <origin xyz="0 0 0" rpy="0 0 0"/>
-        </xacro:inertial_box>
-    </link>
-    <joint name="L_hand_final_joint" type="fixed">
-        <parent link="L_hand_link_x"/>
-        <child link="L_hand_base_link"/>
-        <origin xyz="0 0 0" rpy="0 0 0"/>
-    </joint>
-    <link name="L_hand_base_link">
+    <link name="R_hand_link_x">
+        <xacro:inertial_box mass="0.1" x="0" y="0" z="0">
+            <origin xyz="0 0 0" rpy="0 0 0"/>
+        </xacro:inertial_box>
+    </link>
+    <joint name="R_hand_final_joint" type="fixed">
+        <parent link="R_hand_link_x"/>
+        <child link="R_hand_base_link"/>
+        <origin xyz="0 0 0" rpy="0 0 0"/>
+    </joint>
+    <link name="R_hand_base_link">
         <visual>
             <geometry>
@@ -231,12 +231,12 @@
     </link>
     <!--GRIPPER-->
-    <joint name="L_left_gripper_slide_joint" type="prismatic">
-        <parent link="L_hand_base_link"/>
-        <child link="L_left_gripper_link"/>
+    <joint name="R_left_gripper_slide_joint" type="prismatic">
+        <parent link="R_hand_base_link"/>
+        <child link="R_left_gripper_link"/>
         <origin xyz="0 0.032 -0.035"/>
         <axis xyz="0 -1 0"/>
         <limit effort="10.0" lower="0" upper="0.015" velocity="0.1"/>
     </joint>
-    <link name="L_left_gripper_link">
+    <link name="R_left_gripper_link">
         <visual>
             <geometry>
@@ -254,12 +254,12 @@
         </xacro:inertial_box>
     </link>
-    <joint name="L_right_gripper_slide_joint" type="prismatic">
-        <parent link="L_hand_base_link"/>
-        <child link="L_right_gripper_link"/>
+    <joint name="R_right_gripper_slide_joint" type="prismatic">
+        <parent link="R_hand_base_link"/>
+        <child link="R_right_gripper_link"/>
         <origin xyz="0 -0.032 -0.035"/>
         <axis xyz="0 1 0"/>
         <limit effort="10.0" lower="0" upper="0.015" velocity="0.1"/>
     </joint>
-    <link name="L_right_gripper_link">
+    <link name="R_right_gripper_link">
         <visual>
             <geometry>

File: description/robot.urdf.xacro (robot description, xacro)
@@ -5,3 +5,4 @@
     <xacro:include filename="camera.xacro" />
     <xacro:include filename="left_arm.xacro" />
+    <xacro:include filename="right_arm.xacro" />
 </robot>
