Commit message: Add files via upload

File: description/gazebo_control.xacro (robot description, xacro)
@@ -4,5 +4,6 @@
         <gazebo>
             <plugin name="omni_steering" filename="libgazebo_ros_planar_move.so">
-                <odometry_rate>50.0</odometry_rate>
+                <commandTopic>cmd_vel</commandTopic>
+                <odometry_rate>100.0</odometry_rate>
                 <odometry_frame>odom</odometry_frame>
                 <robot_base_frame>base_link</robot_base_frame>

File: description/left_arm.xacro (robot description, xacro)
@@ -46,5 +46,5 @@
             <origin xyz="0 0 -0.08" rpy="0 0 ${pi/2}"/>
             <geometry>
-                <box size="0.05 0.05 0.2"/>
+                <box size="0.05 0.05 0.3"/>
             </geometry>
             <material name="blue"/>
@@ -139,5 +139,5 @@
             <origin xyz="0 0 -0.08" rpy="0 0 ${pi/2}"/>
             <geometry>
-                <box size="0.05 0.05 0.2"/>
+                <box size="0.05 0.05 0.3"/>
             </geometry>
         </collision>
@@ -230,4 +230,7 @@
         </xacro:inertial_box>
     </link>
+    <gazebo reference="L_hand_base_link">
+        <material>Gazebo/White</material>
+    </gazebo>
     <!--GRIPPER-->
     <joint name="L_left_gripper_slide_joint" type="prismatic">
@@ -277,3 +280,9 @@
         </xacro:inertial_box>
     </link>
+    <gazebo reference="L_left_gripper_link">
+        <material>Gazebo/Red</material>
+    </gazebo>
+    <gazebo reference="L_right_gripper_link">
+        <material>Gazebo/Red</material>
+    </gazebo>
 </robot>

File: description/right_arm.xacro (robot description, xacro)
@@ -46,5 +46,5 @@
             <origin xyz="0 0 -0.08" rpy="0 0 ${pi/2}"/>
             <geometry>
-                <box size="0.05 0.05 0.2"/>
+                <box size="0.05 0.05 0.3"/>
             </geometry>
             <material name="blue"/>
@@ -139,5 +139,5 @@
             <origin xyz="0 0 -0.08" rpy="0 0 ${pi/2}"/>
             <geometry>
-                <box size="0.05 0.05 0.2"/>
+                <box size="0.05 0.05 0.3"/>
             </geometry>
         </collision>
@@ -230,4 +230,7 @@
         </xacro:inertial_box>
     </link>
+    <gazebo reference="R_hand_base_link">
+        <material>Gazebo/White</material>
+    </gazebo>
     <!--GRIPPER-->
     <joint name="R_left_gripper_slide_joint" type="prismatic">
@@ -277,3 +280,9 @@
         </xacro:inertial_box>
     </link>
+    <gazebo reference="R_left_gripper_link">
+        <material>Gazebo/Red</material>
+    </gazebo>
+    <gazebo reference="R_right_gripper_link">
+        <material>Gazebo/Red</material>
+    </gazebo>
 </robot>

File: description/robot.urdf.xacro (robot description, xacro)
@@ -1,7 +1,7 @@
 <?xml version="1.0"?>
 <robot xmlns:xacro="http://www.ros.org/wiki/xacro"  name="robot">
-    <xacro:include filename="robot_core.xacro" />
+    <xacro:include filename="robot_core_Rui.xacro" />
+    <xacro:include filename="depth_camera.xacro" />
     <xacro:include filename="lidar.xacro" />
-    <xacro:include filename="camera.xacro" />
     <xacro:include filename="left_arm.xacro" />
     <xacro:include filename="right_arm.xacro" />

File: description/robot_core.xacro (robot description, xacro)
@@ -15,74 +15,45 @@
         <color rgba="1 0 0 1"/>
     </material>
-    <!--BASE LINK-->
+    <!-- BASE LINK -->
     <link name="base_link">
     </link>
-    <!--CHASSI-->
-    <joint name="chassi_joint" type="fixed">
+    <!-- CHASSIS LINK -->
+    <joint name="chassis_joint" type="fixed">
         <parent link="base_link"/>
-        <child link="chassi_link"/>
-        <origin xyz="0 0 0"/> <!--VIRADO PARA X-->
-        <!--<origin xyz="0 0 0" rpy="0 0 ${pi/2}"/> VIRADO PARA Y-->
+        <child link="chassis"/>
+        <origin xyz="-0.1 0 0"/>
     </joint>
-    <link name="chassi_link">
+    <link name="chassis">
         <visual>
-            <origin xyz="0 0 0.085"/>
+            <origin xyz="0.15 0 0.075"/>
             <geometry>
-                <cylinder radius="0.275" length="0.17"/>
+                <box size="0.3 0.3 0.15"/>
             </geometry>
             <material name="white"/>
         </visual>
         <collision>
-            <origin xyz="0 0 0.085"/>
+            <origin xyz="0.15 0 0.075"/>
             <geometry>
-                <cylinder radius="0.275" length="0.17"/>
+                <box size="0.3 0.3 0.15"/>
             </geometry>
         </collision>
-        <xacro:inertial_cylinder mass="0.1" length="0.17" radius="0.275">
-            <origin xyz="0 0 0.085" rpy="0 0 0"/>
-        </xacro:inertial_cylinder>
+        <xacro:inertial_box mass="0.5" x="0.3" y="0.3" z="0.15">
+            <origin xyz="0.15 0 0.075" rpy="0 0 0"/>
+        </xacro:inertial_box>
     </link>
-    <gazebo reference="chassi_link">
+    <gazebo reference="chassis">
         <material>Gazebo/White</material>
     </gazebo>
-    <!--BODY-->
-    <joint name="body_joint" type="fixed">
-        <parent link="chassi_link"/>
-        <child link="body_link"/>
-        <origin xyz="-0.1 0 0.18" rpy="0 0 0"/>
-    </joint>
-    <link name="body_link">
-        <visual>
-            <origin xyz="0 0 0.55" rpy="0 0 ${pi/2}"/>
-            <geometry>
-                <box size="0.2 0.05 1.1"/>
-            </geometry>
-            <material name="white"/>
-        </visual>
-        <collision>
-            <origin xyz="0 0 0.55" rpy="0 0 ${pi/2}"/>
-            <geometry>
-                <box size="0.2 0.05 1.1"/>
-            </geometry>
-        </collision>
-        <xacro:inertial_box mass="0.1" x="0.2" y="0.05" z="1.1">
-            <origin xyz="0 0 0.55" rpy="0 0 0"/>
-        </xacro:inertial_box>
-    </link>
-    <gazebo reference="body_link">
-        <material>Gazebo/White</material>
-    </gazebo>
-    <!--WHEELS-->
-    <!--LEFT FRONT-->
-    <joint name="left_front_joint" type="continuous">
-        <parent link="chassi_link"/>
-        <child link="left_front_link"/>
-        <origin xyz="0.2 0.2 0" rpy="-${pi/2} 0 -${pi/4}"/>
+    <!-- LEFT WHEEL LINK -->
+    <joint name="left_wheel_joint" type="continuous">
+        <parent link="base_link"/>
+        <child link="left_wheel"/>
+        <origin xyz="0 0.175 0" rpy="-${pi/2} 0 0" />
         <axis xyz="0 0 1"/>
     </joint>
-    <link name="left_front_link">
+    <link name="left_wheel">
         <visual>
             <geometry>
-                <cylinder radius="0.1" length="0.04"/>
+                <cylinder radius="0.05" length="0.04"/>
             </geometry>
             <material name="blue"/>
@@ -90,27 +61,50 @@
         <collision>
             <geometry>
-                <cylinder radius="0.1" length="0.04"/>
+                <cylinder radius="0.05" length="0.04"/>
             </geometry>
         </collision>
-        <xacro:inertial_cylinder mass="0.1" length="0.04" radius="0.1">
+        <xacro:inertial_cylinder mass="0.1" length="0.04" radius="0.05">
             <origin xyz="0 0 0" rpy="0 0 0"/>
         </xacro:inertial_cylinder>
     </link>
-    <gazebo reference="left_front_link">
+    <gazebo reference="left_wheel">
         <material>Gazebo/Blue</material>
-        <mu1 value="0.001"/>
-        <mu2 value="0.001"/>
     </gazebo>
-    <!--LEFT BACK-->
-    <joint name="left_back_joint" type="continuous">
-        <parent link="chassi_link"/>
-        <child link="left_back_link"/>
-        <origin xyz="-0.2 0.2 0" rpy="0 -${pi/2} -${pi/4}"/>
-        <axis xyz="0 0 1"/>
+    <!-- RIGHT WHEEL LINK -->
+    <joint name="right_wheel_joint" type="continuous">
+        <parent link="base_link"/>
+        <child link="right_wheel"/>
+        <origin xyz="0 -0.175 0" rpy="${pi/2} 0 0" />
+        <axis xyz="0 0 -1"/>
     </joint>
-    <link name="left_back_link">
+    <link name="right_wheel">
         <visual>
             <geometry>
-                <cylinder radius="0.1" length="0.04"/>
+                <cylinder radius="0.05" length="0.04"/>
+            </geometry>
+            <material name="blue"/>
+        </visual>
+        <collision>
+            <geometry>
+                <cylinder radius="0.05" length="0.04"/>
+            </geometry>
+        </collision>
+        <xacro:inertial_cylinder mass="0.1" length="0.04" radius="0.05">
+            <origin xyz="0 0 0" rpy="0 0 0"/>
+        </xacro:inertial_cylinder>
+    </link>
+    <gazebo reference="right_wheel">
+        <material>Gazebo/Blue</material>
+    </gazebo>
+    <!-- CASTER WHEEL LINK -->
+    <joint name="caster_wheel_joint" type="fixed">
+        <parent link="chassis"/>
+        <child link="caster_wheel"/>
+        <origin xyz="0.24 0 0"/>
+    </joint>
+    <link name="caster_wheel">
+        <visual>
+            <geometry>
+                <sphere radius="0.05"/>
             </geometry>
             <material name="black"/>
@@ -118,68 +112,12 @@
         <collision>
             <geometry>
-                <cylinder radius="0.1" length="0.04"/>
+                <sphere radius="0.05"/>
             </geometry>
         </collision>
-        <xacro:inertial_cylinder mass="0.1" length="0.04" radius="0.1">
+        <xacro:inertial_sphere mass="0.1" radius="0.05">
             <origin xyz="0 0 0" rpy="0 0 0"/>
-        </xacro:inertial_cylinder>
+        </xacro:inertial_sphere>
     </link>
-    <gazebo reference="left_back_link">
-        <material>Gazebo/Black</material>
-        <mu1 value="0.001"/>
-        <mu2 value="0.001"/>
-    </gazebo>
-    <!--RIGHT FRONT-->
-    <joint name="right_front_joint" type="continuous">
-        <parent link="chassi_link"/>
-        <child link="right_front_link"/>
-        <origin xyz="0.2 -0.2 0" rpy="0 ${pi/2} -${pi/4}"/>
-        <axis xyz="0 0 -1"/>
-    </joint>
-    <link name="right_front_link">
-        <visual>
-            <geometry>
-                <cylinder radius="0.1" length="0.04"/>
-            </geometry>
-            <material name="blue"/>
-        </visual>
-        <collision>
-            <geometry>
-                <cylinder radius="0.1" length="0.04"/>
-            </geometry>
-        </collision>
-        <xacro:inertial_cylinder mass="0.1" length="0.04" radius="0.1">
-            <origin xyz="0 0 0" rpy="0 0 0"/>
-        </xacro:inertial_cylinder>
-    </link>
-    <gazebo reference="right_front_link">
-        <material>Gazebo/Blue</material>
-        <mu1 value="0.001"/>
-        <mu2 value="0.001"/>
-    </gazebo>
-    <!--RIGHT BACK-->
-    <joint name="right_back_joint" type="continuous">
-        <parent link="chassi_link"/>
-        <child link="right_back_link"/>
-        <origin xyz="-0.2 -0.2 0" rpy="${pi/2} 0 -${pi/4}"/>
-        <axis xyz="0 0 -1"/>
-    </joint>
-    <link name="right_back_link">
-        <visual>
-            <geometry>
-                <cylinder radius="0.1" length="0.04"/>
-            </geometry>
-            <material name="black"/>
-        </visual>
-        <collision>
-            <geometry>
-                <cylinder radius="0.1" length="0.04"/>
-            </geometry>
-        </collision>
-        <xacro:inertial_cylinder mass="0.1" length="0.04" radius="0.1">
-            <origin xyz="0 0 0" rpy="0 0 0"/>
-        </xacro:inertial_cylinder>
-    </link>
-    <gazebo reference="right_back_link">
+    <gazebo reference="caster_wheel">
         <material>Gazebo/Black</material>
         <mu1 value="0.001"/>
