Commit message: Add files via upload

File: description/robot_core_Rui.xacro (robot description, xacro)
@@ -17,4 +17,12 @@
     <!--BASE LINK-->
     <link name="base_link">
+    </link>
+    <!--BASE FOOTPRINT LINK-->
+    <joint name="base_footprint_joint" type="fixed">
+        <parent link="base_link"/>
+        <child link="base_footprint"/>
+        <origin xyz="0 0 0" rpy="0 0 0"/>
+    </joint>
+    <link name="base_footprint">
     </link>
     <!--CHASSI-->
@@ -76,5 +84,5 @@
     <!--LEFT FRONT-->
     <joint name="left_front_joint" type="continuous">
-        <parent link="base_link"/>
+        <parent link="chassi_link"/>
         <child link="left_front_link"/>
         <origin xyz="0.2 0.2 0" rpy="-${pi/2} 0 -${pi/4}"/>
@@ -104,5 +112,5 @@
     <!--LEFT BACK-->
     <joint name="left_back_joint" type="continuous">
-        <parent link="base_link"/>
+        <parent link="chassi_link"/>
         <child link="left_back_link"/>
         <origin xyz="-0.2 0.2 0" rpy="0 -${pi/2} -${pi/4}"/>
@@ -132,5 +140,5 @@
     <!--RIGHT FRONT-->
     <joint name="right_front_joint" type="continuous">
-        <parent link="base_link"/>
+        <parent link="chassi_link"/>
         <child link="right_front_link"/>
         <origin xyz="0.2 -0.2 0" rpy="0 ${pi/2} -${pi/4}"/>
@@ -160,5 +168,5 @@
     <!--RIGHT BACK-->
     <joint name="right_back_joint" type="continuous">
-        <parent link="base_link"/>
+        <parent link="chassi_link"/>
         <child link="right_back_link"/>
         <origin xyz="-0.2 -0.2 0" rpy="${pi/2} 0 -${pi/4}"/>
