Commit message: Add files via upload

File: description/robot.urdf.xacro (robot description, xacro)
@@ -2,6 +2,6 @@
 <robot xmlns:xacro="http://www.ros.org/wiki/xacro"  name="robot">
     <xacro:include filename="robot_core_Rui.xacro" />
-    <xacro:include filename="depth_camera.xacro" />
     <xacro:include filename="lidar.xacro" />
+    <xacro:include filename="camera.xacro" />
     <xacro:include filename="left_arm.xacro" />
     <xacro:include filename="right_arm.xacro" />

File: description/robot_core_Rui.xacro (robot description, xacro)
@@ -83,9 +83,8 @@
     <!--WHEELS-->
     <!--LEFT FRONT-->
-    <joint name="left_front_joint" type="continuous">
+    <joint name="left_front_joint" type="fixed">
         <parent link="chassi_link"/>
         <child link="left_front_link"/>
         <origin xyz="0.2 0.2 0" rpy="-${pi/2} 0 -${pi/4}"/>
-        <axis xyz="0 0 1"/>
     </joint>
     <link name="left_front_link">
@@ -111,9 +110,8 @@
     </gazebo>
     <!--LEFT BACK-->
-    <joint name="left_back_joint" type="continuous">
+    <joint name="left_back_joint" type="fixed">
         <parent link="chassi_link"/>
         <child link="left_back_link"/>
         <origin xyz="-0.2 0.2 0" rpy="0 -${pi/2} -${pi/4}"/>
-        <axis xyz="0 0 1"/>
     </joint>
     <link name="left_back_link">
@@ -139,9 +137,8 @@
     </gazebo>
     <!--RIGHT FRONT-->
-    <joint name="right_front_joint" type="continuous">
+    <joint name="right_front_joint" type="fixed">
         <parent link="chassi_link"/>
         <child link="right_front_link"/>
         <origin xyz="0.2 -0.2 0" rpy="0 ${pi/2} -${pi/4}"/>
-        <axis xyz="0 0 -1"/>
     </joint>
     <link name="right_front_link">
@@ -167,9 +164,8 @@
     </gazebo>
     <!--RIGHT BACK-->
-    <joint name="right_back_joint" type="continuous">
+    <joint name="right_back_joint" type="fixed">
         <parent link="chassi_link"/>
         <child link="right_back_link"/>
         <origin xyz="-0.2 -0.2 0" rpy="${pi/2} 0 -${pi/4}"/>
-        <axis xyz="0 0 -1"/>
     </joint>
     <link name="right_back_link">
