Commit message: Add files via upload

File: description/camera.xacro (robot description, xacro)
@@ -4,5 +4,5 @@
         <parent link="body_link"/>
         <child link="camera_link"/>
-        <origin xyz="0 0 1.1" rpy="0 0 0"/>
+        <origin xyz="0.05 0 1.1" rpy="0 0.261 0"/>
     </joint>
     <link name="camera_link">
@@ -24,5 +24,5 @@
         <sensor name="camera" type="camera">
             <pose> 0 0 0 0 0 0 </pose>
-            <visualize>false</visualize>
+            <visualize>true</visualize>
             <update_rate>10</update_rate>
             <camera>

File: description/lidar.xacro (robot description, xacro)
@@ -26,5 +26,5 @@
         <sensor name="laser" type="ray">
             <pose> 0 0 0 0 0 0 </pose>
-            <visualize>true</visualize>
+            <visualize>false</visualize>
             <update_rate>10</update_rate>
             <ray>

File: description/robot_core.xacro (robot description, xacro)
@@ -22,5 +22,6 @@
         <parent link="base_link"/>
         <child link="chassi_link"/>
-        <origin xyz="0 0 0"/>
+        <origin xyz="0 0 0"/> <!--VIRADO PARA X-->
+        <!--<origin xyz="0 0 0" rpy="0 0 ${pi/2}"/> VIRADO PARA Y-->
     </joint>
     <link name="chassi_link">

Commit message: Add files via upload

File: description/camera.xacro (robot description, xacro)
@@ -1,8 +1,10 @@
 <?xml version="1.0"?>
 <robot xmlns:xacro="http://www.ros.org/wiki/xacro">
-    <joint name="camera_joint" type="fixed">
+    <joint name="camera_joint" type="revolute">
         <parent link="body_link"/>
         <child link="camera_link"/>
-        <origin xyz="0.05 0 1.1" rpy="0 0.261 0"/>
+        <origin xyz="0.05 0 1.1" rpy="0 0 0"/>
+        <axis xyz="0 1 0"/>
+        <limit effort="1000.0" lower="0.0" upper="0.548" velocity="0.5"/>
     </joint>
     <link name="camera_link">
@@ -13,4 +15,7 @@
             <material name="red"/>
         </visual>
+        <xacro:inertial_box mass="0.1" x="0.04" y="0.07" z="0.04">
+            <origin xyz="0 0 0" rpy="0 0 0"/>
+        </xacro:inertial_box>
     </link>
     <joint name="camera_optical_joint" type="fixed">

File: description/lidar.xacro (robot description, xacro)
@@ -26,5 +26,5 @@
         <sensor name="laser" type="ray">
             <pose> 0 0 0 0 0 0 </pose>
-            <visualize>false</visualize>
+            <visualize>true</visualize>
             <update_rate>10</update_rate>
             <ray>

Commit message: Add files via upload

File: description/camera.xacro (robot description, xacro)
@@ -4,5 +4,5 @@
         <parent link="body_link"/>
         <child link="camera_link"/>
-        <origin xyz="0.05 0 1.1" rpy="0 0 0"/>
+        <origin xyz="0.045 0 1.12" rpy="0 0 0"/>
         <axis xyz="0 1 0"/>
         <limit effort="1000.0" lower="0.0" upper="0.548" velocity="0.5"/>

Commit message: Add files via upload

File: description/camera.xacro (robot description, xacro)
@@ -1,10 +1,42 @@
 <?xml version="1.0"?>
 <robot xmlns:xacro="http://www.ros.org/wiki/xacro">
-    <joint name="camera_joint" type="revolute">
+    <joint name="neck_joint" type="fixed">
         <parent link="body_link"/>
-        <child link="camera_link"/>
+        <child link="neck_link"/>
         <origin xyz="0.045 0 1.12" rpy="0 0 0"/>
+    </joint>
+    <link name="neck_link">
+        <xacro:inertial_box mass="0.1" x="0" y="0" z="0">
+            <origin xyz="0 0 0" rpy="0 0 0"/>
+        </xacro:inertial_box>
+    </link>
+    <joint name="camera_joint_z" type="revolute">
+        <parent link="neck_link"/>
+        <child link="camera_link_z"/>
+        <origin xyz="0 0 0" rpy="0 0 0"/>
         <axis xyz="0 1 0"/>
         <limit effort="1000.0" lower="0.0" upper="0.548" velocity="0.5"/>
+    </joint>
+    <link name="camera_link_z">
+        <xacro:inertial_box mass="0.1" x="0" y="0" z="0">
+            <origin xyz="0 0 0" rpy="0 0 0"/>
+        </xacro:inertial_box>
+    </link>
+    <joint name="camera_joint_y" type="revolute">
+        <parent link="camera_link_z"/>
+        <child link="camera_link_y"/>
+        <origin xyz="0 0 0" rpy="0 0 0"/>
+        <axis xyz="0 0 1"/>
+        <limit effort="1000.0" lower="-0.548" upper="0.548" velocity="0.5"/>
+    </joint>
+    <link name="camera_link_y">
+        <xacro:inertial_box mass="0.1" x="0" y="0" z="0">
+            <origin xyz="0 0 0" rpy="0 0 0"/>
+        </xacro:inertial_box>
+    </link>
+    <joint name="camera_joint" type="fixed">
+        <parent link="camera_link_y"/>
+        <child link="camera_link"/>
+        <origin xyz="0 0 0" rpy="0 0 0"/>
     </joint>
     <link name="camera_link">

File: description/robot.urdf.xacro (robot description, xacro)
@@ -4,3 +4,4 @@
     <xacro:include filename="lidar.xacro" />
     <xacro:include filename="camera.xacro" />
+    <xacro:include filename="arms.xacro" />
 </robot>

Commit message: Add files via upload

File: description/camera.xacro (robot description, xacro)
@@ -2,7 +2,7 @@
 <robot xmlns:xacro="http://www.ros.org/wiki/xacro">
     <joint name="neck_joint" type="fixed">
-        <parent link="body_link"/>
+        <parent link="upper_body_link"/>
         <child link="neck_link"/>
-        <origin xyz="0.045 0 1.12" rpy="0 0 0"/>
+        <origin xyz="0.045 0 0.5" rpy="0 0 0"/>
     </joint>
     <link name="neck_link">

File: description/depth_camera.xacro (robot description, xacro)
@@ -2,7 +2,7 @@
 <robot xmlns:xacro="http://www.ros.org/wiki/xacro">
     <joint name="neck_joint" type="fixed">
-        <parent link="body_link"/>
+        <parent link="upper_body_link"/>
         <child link="neck_link"/>
-        <origin xyz="0.045 0 1.12" rpy="0 0 0"/>
+        <origin xyz="0.045 0 0.8" rpy="0 0 0"/>
     </joint>
     <link name="neck_link">

File: description/gazebo_control.xacro (robot description, xacro)
@@ -13,4 +13,9 @@
             </plugin>
         </gazebo>
-  </xacro:macro>
+    </xacro:macro>
+    <!-- <gazebo>
+        <plugin name="gazebo_ros_control" filename="libgazebo_ros_control.so">
+            <robotNamespace>robot</robotNamespace>
+        </plugin>
+    </gazebo> -->
 </robot>

File: description/left_arm.xacro (robot description, xacro)
@@ -4,7 +4,7 @@
     <!--SHOULDER-ELBOW-->
     <joint name="L_shoulder_joint" type="fixed">
-        <parent link="body_link"/>
+        <parent link="upper_body_link"/>
         <child link="L_shoulder_aux_link"/>
-        <origin xyz="0.05 0.13 1.05" rpy="0 0 0"/>
+        <origin xyz="0 0.13 0.45" rpy="0 0 0"/>
     </joint>
     <link name="L_shoulder_aux_link">
@@ -44,5 +44,5 @@
     <link name="L_shoulder_link">
         <visual>
-            <origin xyz="0 0 -0.08" rpy="0 0 ${pi/2}"/>
+            <origin xyz="0 0 -0.09" rpy="0 0 ${pi/2}"/>
             <geometry>
                 <box size="0.05 0.05 0.3"/>

File: description/right_arm.xacro (robot description, xacro)
@@ -4,7 +4,7 @@
     <!--SHOULDER-ELBOW-->
     <joint name="R_shoulder_joint" type="fixed">
-        <parent link="body_link"/>
+        <parent link="upper_body_link"/>
         <child link="R_shoulder_aux_link"/>
-        <origin xyz="0.05 -0.13 1.05" rpy="0 0 0"/>
+        <origin xyz="0 -0.13 0.45" rpy="0 0 0"/>
     </joint>
     <link name="R_shoulder_aux_link">
@@ -44,5 +44,5 @@
     <link name="R_shoulder_link">
         <visual>
-            <origin xyz="0 0 -0.08" rpy="0 0 ${pi/2}"/>
+            <origin xyz="0 0 -0.09" rpy="0 0 ${pi/2}"/>
             <geometry>
                 <box size="0.05 0.05 0.3"/>

File: description/robot.urdf.xacro (robot description, xacro)
@@ -4,5 +4,5 @@
     <xacro:include filename="lidar.xacro" />
     <xacro:include filename="camera.xacro" />
-    <xacro:include filename="left_arm.xacro" />
-    <xacro:include filename="right_arm.xacro" />
+    <!--<xacro:include filename="left_arm.xacro" />
+    <xacro:include filename="right_arm.xacro" />-->
 </robot>

File: description/robot_core_Rui.xacro (robot description, xacro)
@@ -47,5 +47,5 @@
             </geometry>
         </collision>
-        <xacro:inertial_cylinder mass="0.1" length="0.17" radius="0.275">
+        <xacro:inertial_cylinder mass="1.0" length="0.17" radius="0.275">
             <origin xyz="0 0 0.085" rpy="0 0 0"/>
         </xacro:inertial_cylinder>
@@ -54,31 +54,84 @@
         <material>Gazebo/White</material>
     </gazebo>
-    <!--BODY-->
-    <joint name="body_joint" type="fixed">
-        <parent link="chassi_link"/>
-        <child link="body_link"/>
-        <origin xyz="-0.1 0 0.18" rpy="0 0 0"/>
-    </joint>
-    <link name="body_link">
-        <visual>
-            <origin xyz="0 0 0.55" rpy="0 0 ${pi/2}"/>
-            <geometry>
-                <box size="0.2 0.05 1.1"/>
+    <!--LOWER BODY 35 +/- 14(junta)-->
+    <joint name="lower_body_joint" type="prismatic">
+        <parent link="base_link"/>
+        <child link="lower_body_link"/>
+        <origin xyz="0 0 0.17" rpy="0 0 0"/>
+        <axis xyz="0 0 1"/>
+        <limit lower="0" upper="0.14" velocity="100" effort="100"/>
+    </joint>
+    <link name="lower_body_link">
+        <visual>
+            <origin xyz="0 0 0.18" rpy="0 0 ${pi/2}"/>
+            <geometry>
+                <box size="0.2 0.05 0.35"/>
             </geometry>
             <material name="white"/>
         </visual>
         <collision>
-            <origin xyz="0 0 0.55" rpy="0 0 ${pi/2}"/>
-            <geometry>
-                <box size="0.2 0.05 1.1"/>
-            </geometry>
-        </collision>
-        <xacro:inertial_box mass="0.1" x="0.2" y="0.05" z="1.1">
-            <origin xyz="0 0 0.55" rpy="0 0 0"/>
+            <origin xyz="0 0 0.18" rpy="0 0 ${pi/2}"/>
+            <geometry>
+                <box size="0.2 0.05 0.35"/>
+            </geometry>
+        </collision>
+        <xacro:inertial_box mass="0.01" x="0.2" y="0.05" z="0.35">
+            <origin xyz="0 0 0.18" rpy="0 0 0"/>
         </xacro:inertial_box>
     </link>
-    <gazebo reference="body_link">
+    <gazebo reference="lower_body_link">
         <material>Gazebo/White</material>
     </gazebo>
+    <!--UPPER BODY 50-->
+    <joint name="upper_body_joint" type="revolute">
+        <parent link="lower_body_link"/>
+        <child link="upper_body_link"/>
+        <origin xyz="0 0 0.355" rpy="0 0 0"/>
+        <axis xyz="0 1 0"/>
+        <!--<limit lower="0.34" upper="1.38" velocity="100" effort="100"/>-->
+        <limit lower="0" upper="1.38" velocity="100" effort="100"/>
+    </joint>
+    <link name="upper_body_link">
+        <visual>
+            <origin xyz="0 0 0.25" rpy="0 0 ${pi/2}"/>
+            <geometry>
+                <box size="0.2 0.05 0.50"/>
+            </geometry>
+            <material name="white"/>
+        </visual>
+        <collision>
+            <origin xyz="0 0 0.25" rpy="0 0 ${pi/2}"/>
+            <geometry>
+                <box size="0.2 0.05 0.50"/>
+            </geometry>
+        </collision>
+        <xacro:inertial_box mass="0.03" x="0.2" y="0.05" z="0.50">
+            <origin xyz="0 0 0.25" rpy="0 0 0"/>
+        </xacro:inertial_box>
+    </link>
+    <gazebo reference="upper_body_link">
+        <material>Gazebo/White</material>
+        <!--<turnGravityOff>true</turnGravityOff>
+        <kp value="1000000.0"/>
+        <kd value="1000000.0"/>
+        <mu1 value="0.001"/>
+        <mu2 value="0.001"/>-->
+    </gazebo>
+    <joint name="aux_rear_box_joint" type="fixed">
+        <parent link="upper_body_link"/>
+        <child link="aux_rear_link"/>
+        <origin xyz="-0.2 0 0.125" rpy="0 0 0"/>
+    </joint>
+     <link name="aux_rear_link">
+        <collision>
+            <origin xyz="0 0 0" rpy="0 0 0"/>
+            <geometry>
+                <box size="0.05 0.05 0.05"/>
+            </geometry>
+        </collision>
+        <xacro:inertial_box mass="0.1" x="0.05" y="0.05" z="0.05">
+            <origin xyz="0 0 0" rpy="0 0 0"/>
+        </xacro:inertial_box>
+    </link>
     <!--WHEELS-->
     <!--LEFT FRONT-->
