Commit message: Add files via upload

File: charmie_bot/description/robot.urdf.xacro (robot description, xacro)
@@ -2,8 +2,8 @@
 <robot xmlns:xacro="http://www.ros.org/wiki/xacro"  name="robot">
     <xacro:include filename="robot_core_Rui.xacro"/>
+    <!-- <xacro:include filename="wheels.xacro"/> -->
+    <xacro:include filename="camera.xacro"/>
     <xacro:include filename="lidar.xacro"/>
-    <xacro:include filename="camera.xacro" />
-    <!--
-    <xacro:include filename="left_arm.xacro" />
+    <!-- <xacro:include filename="left_arm.xacro" />
     <xacro:include filename="right_arm.xacro" /> -->
 </robot>

File: charmie_bot/description/robot_core_Rui.xacro (robot description, xacro)
@@ -57,5 +57,5 @@
         <material>Gazebo/White</material>
     </gazebo>
-    <!--LOWER BODY 35 +/- 14(junta)-->
+    <!--LOWER BODY-->
     <joint name="lower_body_joint" type="prismatic">
         <parent link="base_link"/>
@@ -85,12 +85,13 @@
     <gazebo reference="lower_body_link">
         <material>Gazebo/White</material>
+        <turnGravityOff>true</turnGravityOff>
     </gazebo>
-    <!--UPPER BODY 50-->
-    <joint name="upper_body_joint" type="fixed">
+    <!--UPPER BODY-->
+    <joint name="upper_body_joint" type="revolute">
         <parent link="lower_body_link"/>
         <child link="upper_body_link"/>
         <origin xyz="0 0 0.355" rpy="0 0 0"/>
-        <!-- <axis xyz="0 1 0"/>
-        <limit lower="0.1745" upper="1.2217" velocity="100" effort="100"/> -->
+        <axis xyz="0 1 0"/>
+        <limit lower="0.1745" upper="1.2217" velocity="100" effort="100"/>
     </joint>
     <link name="upper_body_link">
@@ -116,133 +117,4 @@
         <turnGravityOff>true</turnGravityOff>
     </gazebo>
-    <!-- <joint name="aux_rear_box_joint" type="fixed">
-        <parent link="upper_body_link"/>
-        <child link="aux_rear_link"/>
-        <origin xyz="-0.2 0 0.125" rpy="0 0 0"/>
-    </joint>
-     <link name="aux_rear_link">
-        <collision>
-            <origin xyz="0 0 0" rpy="0 0 0"/>
-            <geometry>
-                <box size="0.05 0.05 0.05"/>
-            </geometry>
-        </collision>
-        <xacro:inertial_box mass="0.1" x="0.05" y="0.05" z="0.05">
-            <origin xyz="0 0 0" rpy="0 0 0"/>
-        </xacro:inertial_box>
-    </link> -->
-    <!--WHEELS-->
-    <!--LEFT FRONT-->
-    <joint name="left_front_joint" type="fixed">
-        <parent link="chassi_link"/>
-        <child link="left_front_link"/>
-        <origin xyz="0.2 0.2 0" rpy="-${pi/2} 0 -${pi/4}"/>
-    </joint>
-    <link name="left_front_link">
-        <visual>
-            <geometry>
-                <mesh filename="file://$(find charmie_bot)/description/meshes/omni_wheel.stl" scale="0.001 0.001 0.001"/>
-                <!-- <cylinder radius="0.105" length="0.04"/> -->
-            </geometry>
-            <material name="grey"/>
-        </visual>
-        <collision>
-            <geometry>
-                <cylinder radius="0.105" length="0.04"/>
-            </geometry>
-        </collision>
-        <xacro:inertial_cylinder mass="0.1" length="0.04" radius="0.105">
-            <origin xyz="0 0 0" rpy="0 0 0"/>
-        </xacro:inertial_cylinder>
-    </link>
-    <gazebo reference="left_front_link">
-        <material>Gazebo/Grey</material>
-        <mu1 value="0.001"/>
-        <mu2 value="0.001"/>
-    </gazebo>
-    <!--LEFT BACK-->
-    <joint name="left_back_joint" type="fixed">
-        <parent link="chassi_link"/>
-        <child link="left_back_link"/>
-        <origin xyz="-0.2 0.2 0" rpy="0 -${pi/2} -${pi/4}"/>
-    </joint>
-    <link name="left_back_link">
-        <visual>
-            <geometry>
-                <mesh filename="file://$(find charmie_bot)/description/meshes/omni_wheel.stl" scale="0.001 0.001 0.001"/>
-                <!--<cylinder radius="0.1" length="0.04"/>-->
-            </geometry>
-            <material name="grey"/>
-        </visual>
-        <collision>
-            <geometry>
-                <cylinder radius="0.105" length="0.04"/>
-            </geometry>
-        </collision>
-        <xacro:inertial_cylinder mass="0.1" length="0.04" radius="0.105">
-            <origin xyz="0 0 0" rpy="0 0 0"/>
-        </xacro:inertial_cylinder>
-    </link>
-    <gazebo reference="left_back_link">
-        <material>Gazebo/Grey</material>
-        <mu1 value="0.001"/>
-        <mu2 value="0.001"/>
-    </gazebo>
-    <!--RIGHT FRONT-->
-    <joint name="right_front_joint" type="fixed">
-        <parent link="chassi_link"/>
-        <child link="right_front_link"/>
-        <origin xyz="0.2 -0.2 0" rpy="0 ${pi/2} -${pi/4}"/>
-    </joint>
-    <link name="right_front_link">
-        <visual>
-            <geometry>
-                <mesh filename="file://$(find charmie_bot)/description/meshes/omni_wheel.stl" scale="0.001 0.001 0.001"/>
-                <!--<cylinder radius="0.1" length="0.04"/>-->
-            </geometry>
-            <material name="grey"/>
-        </visual>
-        <collision>
-            <geometry>
-                <cylinder radius="0.105" length="0.04"/>
-            </geometry>
-        </collision>
-        <xacro:inertial_cylinder mass="0.1" length="0.04" radius="0.105">
-            <origin xyz="0 0 0" rpy="0 0 0"/>
-        </xacro:inertial_cylinder>
-    </link>
-    <gazebo reference="right_front_link">
-        <material>Gazebo/Grey</material>
-        <mu1 value="0.001"/>
-        <mu2 value="0.001"/>
-    </gazebo>
-    <!--RIGHT BACK-->
-    <joint name="right_back_joint" type="fixed">
-        <parent link="chassi_link"/>
-        <child link="right_back_link"/>
-        <origin xyz="-0.2 -0.2 0" rpy="${pi/2} 0 -${pi/4}"/>
-    </joint>
-    <link name="right_back_link">
-        <visual>
-            <geometry>
-                <mesh filename="file://$(find charmie_bot)/description/meshes/omni_wheel.stl" scale="0.001 0.001 0.001"/>
-                <!--<cylinder radius="0.1" length="0.04"/>-->
-            </geometry>
-            <material name="grey"/>
-        </visual>
-        <collision>
-            <geometry>
-                <cylinder radius="0.105" length="0.04"/>
-            </geometry>
-        </collision>
-        <xacro:inertial_cylinder mass="0.1" length="0.04" radius="0.105">
-            <origin xyz="0 0 0" rpy="0 0 0"/>
-        </xacro:inertial_cylinder>
-    </link>
-    <gazebo reference="right_back_link">
-        <material>Gazebo/Grey</material>
-        <mu1 value="0.001"/>
-        <mu2 value="0.001"/>
-    </gazebo>
     <xacro:ros2_control_gazebo/>
 </robot>

File: charmie_bot/description/ros2_control.xacro (robot description, xacro)
@@ -6,8 +6,28 @@
                 <plugin>gazebo_ros2_control/GazeboSystem</plugin>
             </hardware>
+            <!--CAMERA-->
+            <joint name="camera_joint_y">
+                <command_interface name="position">
+                    <param name="min">-0.548</param>
+                    <param name="max">0.548</param>
+                </command_interface>
+                <state_interface name="position"/>
+                <state_interface name="velocity"/>
+                <state_interface name="effort"/>
+            </joint>
             <joint name="camera_joint_z">
                 <command_interface name="position">
                     <param name="min">-0.548</param>
                     <param name="max">0.548</param>
+                </command_interface>
+                <state_interface name="position"/>
+                <state_interface name="velocity"/>
+                <state_interface name="effort"/>
+            </joint>
+            <!--BODY-->
+            <joint name="upper_body_joint">
+                <command_interface name="position">
+                    <param name="min">0.1745</param>
+                    <param name="max">1.2217</param>
                 </command_interface>
                 <state_interface name="position"/>
